File: yusynth_vco.sch (EAGLE design)
At the start: 100 parts, among them IC2 LM311N, J2 LINEAR FM, J3 SOFT SYNC IN, J4 HARD SYNC IN, Q1 J111, T1 220K, T2 22K, T3 10K, T4 10K, U1 7812L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

Commit message: actually distribute accross sheets
Parts:
- added U5: TL074P, linear:TL074P
Connections:
- net GNDA: now also U5B.+IN, U5C.+IN; no longer U7B.+IN, U7C.+IN
- net N$22: now also U5B.OUT; no longer U7B.OUT
- net N$24: now also U5B.-IN; no longer U7B.-IN
- net N$25: now also U5C.-IN; no longer U7C.-IN
- net N$29: now also U5D.-IN; no longer U7D.-IN
- net N$30: now also U5D.+IN; no longer U7D.+IN
- net SINE_OUT: now also U5D.OUT; no longer U7D.OUT
- net TRI_OUT: now also U5C.OUT; no longer U7C.OUT
